File: LSF0204-Breakout.brd (EAGLE design)
At the start: 15.7 x 16.2 mm, 15 parts, among them U1 LSF0204

Commit message: Updated schematics and aesthetics.
Parts:
- C1, C2: value (none) -> 0.1uF
- R9: value (none) -> 10k
Changed lines of the file:
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@@
 <layer number="25" name="tNames" color="7" fill="1" visible="yes" active="yes"/>
 <layer number="26" name="bNames" color="7" fill="1" visible="yes" active="yes"/>
-<layer number="27" name="tValues" color="7" fill="1" visible="yes" active="yes"/>
-<layer number="28" name="bValues" color="7" fill="1" visible="yes" active="yes"/>
+<layer number="27" name="tValues" color="7" fill="1" visible="no" active="yes"/>
+<layer number="28" name="bValues" color="7" fill="1" visible="no" active="yes"/>
 <layer number="29" name="tStop" color="7" fill="3" visible="yes" active="yes"/>
 <layer number="30" name="bStop" color="7" fill="6" visible="yes" active="yes"/>
@@
 <elements>
 <element name="U1" library="Fra" package="TSSOP_14" value="LSF0204" x="-0.005" y="-0.005"/>
-<element name="R9" library="SparkFun-Passives" package="0805" value="" x="4.44" y="-0.005" smashed="yes" rot="R270">
+<element name="R9" library="SparkFun-Passives" package="0805" value="10k" x="4.44" y="-0.005" smashed="yes" rot="R270">
 <attribute name="VALUE" x="3.043" y="1.011" size="0.4064" layer="27" rot="R270"/>
 </element>
@@
 <attribute name="VALUE" x="-7.625" y="3.043" size="1.27" layer="27" font="vector"/>
 </element>
-<element name="C1" library="SparkFun-Passives" package="0805" value="" x="-6.355" y="-0.005" smashed="yes" rot="R90">
+<element name="C1" library="SparkFun-Passives" package="0805" value="0.1uF" x="-6.355" y="-0.005" smashed="yes" rot="R90">
 <attribute name="VALUE" x="-4.958" y="-1.021" size="0.4064" layer="27" rot="R90"/>
 </element>
-<element name="C2" library="SparkFun-Passives" package="0805" value="" x="-4.45" y="-0.005" smashed="yes" rot="R270">
+<element name="C2" library="SparkFun-Passives" package="0805" value="0.1uF" x="-4.45" y="-0.005" smashed="yes" rot="R270">
 <attribute name="VALUE" x="-5.847" y="1.011" size="0.4064" layer="27" rot="R270"/>
 </element>
